Commit message: URDF LINK

File: tx90_moveit_config/urdf/CFRP.urdf (robot description, URDF)
Before this commit: robot mobile_robot, 2 links, 0 joints
Links:
- removed link base_footprint
- removed link base_link
- added link babbbbse_link, mass 0.5; collision box size=0.1 0.1 0.01; visual box size=0.1 0.1 0.01
- added link top_part
Joints:
- added joint $cfrp_joint: type fixed, parent babbbbse_link, child top_part, origin xyz=0 0 0 rpy=0 0 0
