Commit message: new cfrp model

File: test_bed/urdf/freeform_cfrp.urdf (robot description, URDF)
Before this commit: robot test_bed, 1 links, 0 joints
Links:
- removed link base_link
- added link freeform_cfrp, mass 0.1; collision mesh filename=package://freeform_cfrp/meshes/freeform_cfrp.STL; visual mesh filename=package://freeform_cfrp/meshes/freeform_cfrp.STL
