Commit message: pcd file added

File: staubli_tx90_gazebo/urdf/tx90_macro.xacro (robot description, xacro)
@@ -100,9 +100,9 @@
     <turnGravityOff>true</turnGravityOff>
   </gazebo>
-  <gazebo reference="${prefix}cfrp_base">
-    <material>Gazebo/Orange</material>
-  </gazebo>
   <gazebo reference="${prefix}bed_base">
     <material>Gazebo/Grey</material>
+  </gazebo>
+  <gazebo reference="${prefix}PVS_1000_chuck">
+    <material>Gazebo/light_grey</material>
   </gazebo>
   <!-- ros_control plugin -->

File: staubli_tx90_support/urdf/cfrp_macro.xacro (robot description, xacro)
@@ -6,5 +6,7 @@
       <visual>
         <origin xyz="0 0 0" rpy="0 0 0"/>
-        <material name="orange"/>
+        <material name="light black">
+          <color rgba = "5.0 0 0 0.7"/>
+        </material>
         <geometry>
           <mesh
@@ -25,5 +27,5 @@
     </link>
     <gazebo reference="${prefix}cfrp_base">
-      <material>Gazebo/Orange</material>
+      <material>Gazebo/Grey</material>
     </gazebo>
   </xacro:macro>

File: staubli_tx90_support/urdf/tx90_macro.xacro (robot description, xacro)
@@ -187,8 +187,10 @@
     <visual>
       <origin xyz="0.0 0.07 0.0"/>
-      <material name="orange"/>
-      <geometry>
-        <mesh filename="package://test_bed/meshes/PVS_1000_chuck.STL" />
-      </geometry>
+      <geometry>
+        <mesh filename="package://test_bed/meshes/PVS_1000_chuck.dae" />
+      </geometry>
+      <material name="light_grey">
+        <color rgba="10.0 0.0 0.0 0.5" />
+      </material>
     </visual>
     <collision>

Commit message: little update

File: staubli_tx90_gazebo/urdf/tx90_macro.xacro (robot description, xacro)
@@ -100,6 +100,6 @@
     <turnGravityOff>true</turnGravityOff>
   </gazebo>
-  <gazebo reference="${prefix}bed_base">
-    <material>Gazebo/Grey</material>
+  <gazebo reference="${prefix}bed_color">
+    <material>Gazebo/Yellow</material>
   </gazebo>
   <gazebo reference="${prefix}PVS_1000_chuck">

File: staubli_tx90_support/urdf/tx90_macro.xacro (robot description, xacro)
@@ -235,4 +235,7 @@
     </inertial>
     <visual>
+      <material name="bed_color">
+        <color rgba="0.79216 0.81961 0.93333 1" />
+      </material>
       <origin xyz="0 0 0" rpy="0 0 0" />
       <geometry>
@@ -241,6 +244,6 @@
       </geometry>
       <material
-        name="">
-        <color nrgba="0.52549 0.52549 0.52549 1" />
+        name="bed_color">
+        <color nrgba="0.79216 0.81961 0.93333 1" />
       </material>
     </visual>
