Commit message: chuck added

File: staubli_tx90_gazebo/urdf/tx90.xacro (robot description, xacro)
@@ -17,7 +17,7 @@
     <origin xyz="-0.278 -0.033 0.75" rpy="0.0 0.0 0.0" />
   </joint>
-  <joint name="bed_base-cfrp_base-fixed" type="fixed">
+  <joint name="bed_base-PVS_1000_chuck-fixed" type="fixed">
     <parent link="bed_base"/>
-    <child link="cfrp_base"/>
+    <child link="PVS_1000_chuck"/>
     <origin xyz="0.45 0.0 0.75" rpy="0.0 0.0 0.0" />
   </joint>

File: staubli_tx90_support/urdf/tx90_macro.xacro (robot description, xacro)
@@ -184,21 +184,21 @@
       </inertial>
   </link>
-  <link name="${prefix}cfrp_base">
+  <link name="${prefix}PVS_1000_chuck">
     <visual>
-      <origin xyz="0 0 0" rpy="0 0 0"/>
+      <origin xyz="0.0 0.0 0.0"/>
       <material name="orange"/>
       <geometry>
-          <box size="0.1 0.1 0.0025"/>
+        <mesh filename="package://test_bed/meshes/PVS_1000_chuck.STL" />
       </geometry>
     </visual>
     <collision>
         <geometry>
-            <box size="0.1 0.1 0.0025"/>
+            <mesh filename="package://test_bed/meshes/PVS_1000_chuck.STL" />
         </geometry>
         <origin xyz="0 0 0" rpy="0 0 0"/>
     </collision>
     <inertial>
-        <mass value="1"/>
-        <inertia ixx="1.0" ixy="0.0" ixz="0.0" iyy="1.0" iyz="0.0" izz="1.0"/>
+        <mass value="3.4926" />/>
+        <inertia ixx="0.039719" ixy="0.0" ixz="0.0" iyy="0.006139" iyz="-0.00014653" izz="0.038919"/>
     </inertial>
   </link>

Commit message: cylinder shape cfrp added

File: staubli_tx90_gazebo/urdf/tx90.xacro (robot description, xacro)
@@ -20,5 +20,10 @@
     <parent link="bed_base"/>
     <child link="PVS_1000_chuck"/>
-    <origin xyz="0.45 0.0 0.75" rpy="0.0 0.0 0.0" />
+    <origin xyz="0.45 -0.2 0.75" rpy="0.0 0.0 0.0" />
   </joint>
+<!--   <joint name="PVS_1000_chuck_surface_cfrp-fixed" type="fixed">
+    <parent link="PVS_1000_chuck"/>
+    <child link="surface_cfrp"/>
+    <origin xyz="0.0 0.0 0.1" rpy="0.0 0.0 0.0" />
+  </joint> -->
 </robot>

File: staubli_tx90_support/urdf/cfrp_macro.xacro (robot description, xacro)
@@ -8,16 +8,18 @@
         <material name="orange"/>
         <geometry>
-            <box size="0.1 0.1 0.0025"/>
+          <mesh
+            filename="package://test_bed/meshes/surface_cfrp.STL" />
         </geometry>
       </visual>
       <collision>
           <geometry>
-              <box size="0.1 0.1 0.0025"/>
+            <mesh
+              filename="package://test_bed/meshes/surface_cfrp.STL" />
           </geometry>
           <origin xyz="0 0 0" rpy="0 0 0"/>
       </collision>
       <inertial>
-          <mass value="1"/>
-          <inertia ixx="1.0" ixy="0.0" ixz="0.0" iyy="1.0" iyz="0.0" izz="1.0"/>
+          <mass value="0.18618"/>
+          <inertia ixx="0.00061682" ixy="0.0" ixz="0.0" iyy="0.00045111" iyz="0.0" izz="0.00087324"/>
       </inertial>
     </link>

File: staubli_tx90_support/urdf/tx90_macro.xacro (robot description, xacro)
@@ -186,5 +186,5 @@
   <link name="${prefix}PVS_1000_chuck">
     <visual>
-      <origin xyz="0.0 0.0 0.0"/>
+      <origin xyz="0.0 0.07 0.0"/>
       <material name="orange"/>
       <geometry>
@@ -203,4 +203,25 @@
     </inertial>
   </link>
+  <!-- <link name="${prefix}surface_cfrp">
+    <visual>
+      <origin xyz="0.0 0.0 0.0"/>
+      <material name="orange">
+        <color rgba="0.79216 0.81961 0.93333 1" />
+      </material>
+      <geometry>
+        <mesh filename="package://test_bed/meshes/surface_cfrp.STL" />
+      </geometry>
+    </visual>
+    <collision>
+        <geometry>
+            <mesh filename="package://test_bed/meshes/surface_cfrp.STL" />
+        </geometry>
+        <origin xyz="0 0 0" rpy="0 0 0"/>
+    </collision>
+    <inertial>
+        <mass value="3.4926" />/>
+        <inertia ixx="0.039719" ixy="0.0" ixz="0.0" iyy="0.006139" iyz="-0.00014653" izz="0.038919"/>
+    </inertial>
+  </link> -->
   <link name="${prefix}bed_base">
     <inertial>

File: test_bed/urdf/surface_cfrp.urdf (robot description, URDF)
Before this commit: robot test_bed, 1 links, 0 joints
Links:
- removed link base_link
- added link surface_cfrp, mass 0.18618; collision mesh filename=package://surface_cfrp/meshes/surface_cfrp.STL; visual mesh filename=package://surface_cfrp/meshes/surface_cfrp.STL

Commit message: position adjustment

File: staubli_tx90_gazebo/urdf/tx90.xacro (robot description, xacro)
@@ -10,15 +10,15 @@
     <parent link="world"/>
     <child link="bed_base"/>
-    <origin xyz="0.0 0.0 0.0" rpy="0.0 0.0 0.0" />
+    <origin xyz="0.278 0.033 0.0" rpy="0.0 0.0 0.0" />
   </joint>
   <joint name="bed_base-base_link-fixed" type="fixed">
     <parent link="bed_base"/>
     <child link="base_link"/>
-    <origin xyz="-0.278 -0.033 0.75" rpy="0.0 0.0 0.0" />
+    <origin xyz="-0.278 -0.033 0.73" rpy="0.0 0.0 0.0" />
   </joint>
   <joint name="bed_base-PVS_1000_chuck-fixed" type="fixed">
     <parent link="bed_base"/>
     <child link="PVS_1000_chuck"/>
-    <origin xyz="0.45 -0.2 0.75" rpy="0.0 0.0 0.0" />
+    <origin xyz="0.45 -0.2 0.73" rpy="0.0 0.0 0.0" />
   </joint>
 <!--   <joint name="PVS_1000_chuck_surface_cfrp-fixed" type="fixed">

File: staubli_tx90_support/urdf/tx90_macro.xacro (robot description, xacro)
@@ -327,5 +327,5 @@
     <link name="${prefix}tool_tip_link" />
     <joint name="${prefix}flange-tool0" type="fixed">
-      <origin xyz="0.15 0 0.15" rpy="0 0 0" />
+      <origin xyz="0.191 0 0.1027" rpy="0 0 0" />
       <parent link="${prefix}tool_link" />
       <child link="${prefix}tool_tip_link" />

Commit message: urdf changed

File: staubli_tx90_gazebo/urdf/tx90.xacro (robot description, xacro)
@@ -22,4 +22,11 @@
     <origin xyz="0.45 -0.2 0.73" rpy="0.0 0.0 0.0" />
   </joint>
+<!--   <joint name="dummy_camera_joint" type="fixed">
+    <axis xyz="0 0 0" />
+    <origin xyz="0 0 0" rpy="0 0 0"/>
+    <parent link="camera_link"/>
+    <child link="dummy_camera_link"/>
+  </joint>  -->
+      <!--<origin xyz="0.0149 0.0275 0" rpy="${M_PI/2} 0 ${M_PI/2}"/>-->
 <!--   <joint name="PVS_1000_chuck_surface_cfrp-fixed" type="fixed">
     <parent link="PVS_1000_chuck"/>

Commit message: overall update

File: staubli_tx90_gazebo/urdf/tx90.xacro (robot description, xacro)
@@ -17,16 +17,9 @@
     <origin xyz="-0.278 -0.033 0.73" rpy="0.0 0.0 0.0" />
   </joint>
-  <joint name="bed_base-PVS_1000_chuck-fixed" type="fixed">
+<!--   <joint name="bed_base-PVS_1000_chuck-fixed" type="fixed">
     <parent link="bed_base"/>
     <child link="PVS_1000_chuck"/>
     <origin xyz="0.45 -0.2 0.73" rpy="0.0 0.0 0.0" />
-  </joint>
-<!--   <joint name="dummy_camera_joint" type="fixed">
-    <axis xyz="0 0 0" />
-    <origin xyz="0 0 0" rpy="0 0 0"/>
-    <parent link="camera_link"/>
-    <child link="dummy_camera_link"/>
-  </joint>  -->
-      <!--<origin xyz="0.0149 0.0275 0" rpy="${M_PI/2} 0 ${M_PI/2}"/>-->
+  </joint> -->
 <!--   <joint name="PVS_1000_chuck_surface_cfrp-fixed" type="fixed">
     <parent link="PVS_1000_chuck"/>

File: staubli_tx90_support/urdf/cfrp_macro.xacro (robot description, xacro)
@@ -11,6 +11,5 @@
         <geometry>
           <mesh
-            filename="package://test_bed/meshes/freeform_cfrp.STL" />
-            <!-- filename="package://test_bed/meshes/surface_cfrp.STL" /> -->
+            filename="package://test_bed/meshes/surface_cfrp.STL" />
         </geometry>
       </visual>
@@ -18,6 +17,5 @@
           <geometry>
             <mesh
-              filename="package://test_bed/meshes/freeform_cfrp.STL" />
-              <!-- filename="package://test_bed/meshes/surface_cfrp.STL" /> -->
+              filename="package://test_bed/meshes/surface_cfrp.STL" />
           </geometry>
           <origin xyz="0 0 0" rpy="0 0 0"/>

File: staubli_tx90_support/urdf/tx90_macro.xacro (robot description, xacro)
@@ -184,5 +184,5 @@
       </inertial>
   </link>
-  <link name="${prefix}PVS_1000_chuck">
+<!--   <link name="${prefix}PVS_1000_chuck">
     <visual>
       <origin xyz="0.0 0.07 0.0"/>
@@ -204,5 +204,5 @@
         <inertia ixx="0.039719" ixy="0.0" ixz="0.0" iyy="0.006139" iyz="-0.00014653" izz="0.038919"/>
     </inertial>
-  </link>
+  </link> -->
   <!-- <link name="${prefix}surface_cfrp">
     <visual>
@@ -328,5 +328,5 @@
     <link name="${prefix}tool_tip_link" />
     <joint name="${prefix}flange-tool0" type="fixed">
-      <origin xyz="0.165816 -0.01998 0.1027" rpy="0 0 0" />
+      <origin xyz="0.191 0 0.1027" rpy="0 0 0" />
       <parent link="${prefix}tool_link" />
       <child link="${prefix}tool_tip_link" />
@@ -334,6 +334,6 @@
     <!--D435 -->
   <xacro:include filename="$(find realsense2_description)/urdf/_d435.urdf.xacro" />
-  <xacro:sensor_d435 parent="tool_link">
-        <origin xyz="0.13 0 0.034" rpy="0 ${pi} ${pi}"/>
+  <xacro:sensor_d435 parent="tool_link" use_nominal_extrinsics="$(arg use_nominal_extrinsics)">
+        <origin xyz="0.13 0 0.057" rpy="0 ${pi} ${pi}"/>
     </xacro:sensor_d435>
   </xacro:macro>

Commit message: path planner

File: staubli_tx90_gazebo/urdf/tx90.xacro (robot description, xacro)
@@ -17,9 +17,9 @@
     <origin xyz="-0.278 -0.033 0.73" rpy="0.0 0.0 0.0" />
   </joint>
-<!--   <joint name="bed_base-PVS_1000_chuck-fixed" type="fixed">
+  <joint name="bed_base-PVS_1000_chuck-fixed" type="fixed">
     <parent link="bed_base"/>
     <child link="PVS_1000_chuck"/>
     <origin xyz="0.45 -0.2 0.73" rpy="0.0 0.0 0.0" />
-  </joint> -->
+  </joint>
 <!--   <joint name="PVS_1000_chuck_surface_cfrp-fixed" type="fixed">
     <parent link="PVS_1000_chuck"/>

File: staubli_tx90_support/urdf/tx90_macro.xacro (robot description, xacro)
@@ -184,5 +184,5 @@
       </inertial>
   </link>
-<!--   <link name="${prefix}PVS_1000_chuck">
+  <link name="${prefix}PVS_1000_chuck">
     <visual>
       <origin xyz="0.0 0.07 0.0"/>
@@ -204,5 +204,5 @@
         <inertia ixx="0.039719" ixy="0.0" ixz="0.0" iyy="0.006139" iyz="-0.00014653" izz="0.038919"/>
     </inertial>
-  </link> -->
+  </link>
   <!-- <link name="${prefix}surface_cfrp">
     <visual>

Commit message: overall change

File: staubli_tx90_gazebo/urdf/tx90.xacro (robot description, xacro)
@@ -17,9 +17,9 @@
     <origin xyz="-0.278 -0.033 0.73" rpy="0.0 0.0 0.0" />
   </joint>
-  <joint name="bed_base-PVS_1000_chuck-fixed" type="fixed">
+<!--   <joint name="bed_base-PVS_1000_chuck-fixed" type="fixed">
     <parent link="bed_base"/>
     <child link="PVS_1000_chuck"/>
     <origin xyz="0.45 -0.2 0.73" rpy="0.0 0.0 0.0" />
-  </joint>
+  </joint> -->
 <!--   <joint name="PVS_1000_chuck_surface_cfrp-fixed" type="fixed">
     <parent link="PVS_1000_chuck"/>

File: staubli_tx90_support/urdf/tx90_macro.xacro (robot description, xacro)
@@ -184,5 +184,5 @@
       </inertial>
   </link>
-  <link name="${prefix}PVS_1000_chuck">
+<!--   <link name="${prefix}PVS_1000_chuck">
     <visual>
       <origin xyz="0.0 0.07 0.0"/>
@@ -204,5 +204,5 @@
         <inertia ixx="0.039719" ixy="0.0" ixz="0.0" iyy="0.006139" iyz="-0.00014653" izz="0.038919"/>
     </inertial>
-  </link>
+  </link> -->
   <!-- <link name="${prefix}surface_cfrp">
     <visual>
@@ -326,13 +326,13 @@
     </joint>
     <!-- ROS-Industrial 'tool0' frame: all-zeros tool frame -->
-    <link name="${prefix}tool_tip_link" />
+    <link name="${prefix}tool0" />
     <joint name="${prefix}flange-tool0" type="fixed">
       <origin xyz="0.191 0 0.1027" rpy="0 0 0" />
       <parent link="${prefix}tool_link" />
-      <child link="${prefix}tool_tip_link" />
+      <child link="${prefix}tool0" />
     </joint>
     <!--D435 -->
   <xacro:include filename="$(find realsense2_description)/urdf/_d435.urdf.xacro" />
-  <xacro:sensor_d435 parent="tool_link" use_nominal_extrinsics="$(arg use_nominal_extrinsics)">
+  <xacro:sensor_d435 parent="tool_link">
         <origin xyz="0.13 0 0.057" rpy="0 ${pi} ${pi}"/>
     </xacro:sensor_d435>

Commit message: controller takes to long error solve

File: staubli_tx90_gazebo/urdf/tx90.xacro (robot description, xacro)
@@ -7,19 +7,20 @@
   <!-- Fix robot to Gazebo world -->
   <link name="world"/>
-  <joint name="world-bed_base-fixed" type="fixed">
+<!--   <joint name="world-bed_base-fixed" type="fixed">
     <parent link="world"/>
     <child link="bed_base"/>
     <origin xyz="0.278 0.033 0.0" rpy="0.0 0.0 0.0" />
+  </joint> -->
+  <joint name="world-base_link-fixed" type="fixed">
+    <parent link="world"/>
+    <child link="base_link"/>
+    <!-- <origin xyz="-0.278 -0.033 0.73" rpy="0.0 0.0 0.0" /> -->
+    <origin xyz="0.0 0.0 0.0" rpy="0.0 0.0 0.0" />
   </joint>
-  <joint name="bed_base-base_link-fixed" type="fixed">
-    <parent link="bed_base"/>
-    <child link="base_link"/>
-    <origin xyz="-0.278 -0.033 0.73" rpy="0.0 0.0 0.0" />
-  </joint>
-  <joint name="bed_base-PVS_1000_chuck-fixed" type="fixed">
+<!--   <joint name="bed_base-PVS_1000_chuck-fixed" type="fixed">
     <parent link="bed_base"/>
     <child link="PVS_1000_chuck"/>
     <origin xyz="0.45 -0.2 0.73" rpy="0.0 0.0 0.0" />
-  </joint>
+  </joint> -->
 <!--   <joint name="PVS_1000_chuck_surface_cfrp-fixed" type="fixed">
     <parent link="PVS_1000_chuck"/>

File: staubli_tx90_support/urdf/tx90_macro.xacro (robot description, xacro)
@@ -184,5 +184,5 @@
       </inertial>
   </link>
-  <link name="${prefix}PVS_1000_chuck">
+<!--   <link name="${prefix}PVS_1000_chuck">
     <visual>
       <origin xyz="0.0 0.07 0.0"/>
@@ -197,25 +197,4 @@
         <geometry>
             <mesh filename="package://test_bed/meshes/PVS_1000_chuck.STL" />
-        </geometry>
-        <origin xyz="0 0 0" rpy="0 0 0"/>
-    </collision>
-    <inertial>
-        <mass value="3.4926" />/>
-        <inertia ixx="0.039719" ixy="0.0" ixz="0.0" iyy="0.006139" iyz="-0.00014653" izz="0.038919"/>
-    </inertial>
-  </link>
-  <!-- <link name="${prefix}surface_cfrp">
-    <visual>
-      <origin xyz="0.0 0.0 0.0"/>
-      <material name="orange">
-        <color rgba="0.79216 0.81961 0.93333 1" />
-      </material>
-      <geometry>
-        <mesh filename="package://test_bed/meshes/surface_cfrp.STL" />
-      </geometry>
-    </visual>
-    <collision>
-        <geometry>
-            <mesh filename="package://test_bed/meshes/surface_cfrp.STL" />
         </geometry>
         <origin xyz="0 0 0" rpy="0 0 0"/>
@@ -226,5 +205,26 @@
     </inertial>
   </link> -->
-  <link name="${prefix}bed_base">
+  <!-- <link name="${prefix}surface_cfrp">
+    <visual>
+      <origin xyz="0.0 0.0 0.0"/>
+      <material name="orange">
+        <color rgba="0.79216 0.81961 0.93333 1" />
+      </material>
+      <geometry>
+        <mesh filename="package://test_bed/meshes/surface_cfrp.STL" />
+      </geometry>
+    </visual>
+    <collision>
+        <geometry>
+            <mesh filename="package://test_bed/meshes/surface_cfrp.STL" />
+        </geometry>
+        <origin xyz="0 0 0" rpy="0 0 0"/>
+    </collision>
+    <inertial>
+        <mass value="3.4926" />/>
+        <inertia ixx="0.039719" ixy="0.0" ixz="0.0" iyy="0.006139" iyz="-0.00014653" izz="0.038919"/>
+    </inertial>
+  </link> -->
+<!--   <link name="${prefix}bed_base">
     <inertial>
       <origin xyz="0.062333 0.11301 0.77365" rpy="0 0 0" />
@@ -255,5 +255,5 @@
       </geometry>
     </collision>
-  </link>
+  </link> -->
     <!-- joints: main serial chain -->
     <joint name="${prefix}joint_1" type="revolute">
@@ -331,5 +331,5 @@
     <link name="${prefix}tool0" />
     <joint name="${prefix}flange-tool0" type="fixed">
-      <origin xyz="0.191 0 0.1027" rpy="0 0 0" />
+      <origin xyz="0.17295 0.0034 0.103" rpy="0 0 0" />
       <parent link="${prefix}tool_link" />
       <child link="${prefix}tool0" />
@@ -338,5 +338,5 @@
   <xacro:include filename="$(find realsense2_description)/urdf/_d435.urdf.xacro" />
   <xacro:sensor_d435 parent="tool_link" use_nominal_extrinsics="$(arg use_nominal_extrinsics)">
-        <origin xyz="0.13 0 0.057" rpy="0 ${pi} ${pi}"/>
+        <origin xyz="0.186 0.00 -0.006" rpy="${pi} ${pi} ${pi}"/>
     </xacro:sensor_d435>
   </xacro:macro>
