Commit message: tf fixed

File: staubli_tx90_support/urdf/tx90_macro.xacro (robot description, xacro)
@@ -311,4 +311,5 @@
       <parent link="${prefix}base_link"/>
       <child link="${prefix}base"/>
+      <axis xyz="0 0 0"/>
     </joint>
     <!-- ROS-Industrial 'flange' frame: attachment point for EEF models -->

Commit message: tool position changed

File: staubli_tx90_support/urdf/tx90_macro.xacro (robot description, xacro)
@@ -328,5 +328,5 @@
     <link name="${prefix}tool_tip_link" />
     <joint name="${prefix}flange-tool0" type="fixed">
-      <origin xyz="0.191 0 0.1027" rpy="0 0 0" />
+      <origin xyz="0.165816 -0.01998 0.1027" rpy="0 0 0" />
       <parent link="${prefix}tool_link" />
       <child link="${prefix}tool_tip_link" />
@@ -335,5 +335,5 @@
   <xacro:include filename="$(find realsense2_description)/urdf/_d435.urdf.xacro" />
   <xacro:sensor_d435 parent="tool_link">
-        <origin xyz="0.13 0 0.057" rpy="0 ${pi} ${pi}"/>
+        <origin xyz="0.13 0 0.034" rpy="0 ${pi} ${pi}"/>
     </xacro:sensor_d435>
   </xacro:macro>

Commit message: code cleanup

File: staubli_tx90_support/urdf/tx90_macro.xacro (robot description, xacro)
@@ -184,5 +184,5 @@
       </inertial>
   </link>
-<!--   <link name="${prefix}PVS_1000_chuck">
+  <link name="${prefix}PVS_1000_chuck">
     <visual>
       <origin xyz="0.0 0.07 0.0"/>
@@ -204,5 +204,5 @@
         <inertia ixx="0.039719" ixy="0.0" ixz="0.0" iyy="0.006139" iyz="-0.00014653" izz="0.038919"/>
     </inertial>
-  </link> -->
+  </link>
   <!-- <link name="${prefix}surface_cfrp">
     <visual>
@@ -337,5 +337,5 @@
     <!--D435 -->
   <xacro:include filename="$(find realsense2_description)/urdf/_d435.urdf.xacro" />
-  <xacro:sensor_d435 parent="tool_link">
+  <xacro:sensor_d435 parent="tool_link" use_nominal_extrinsics="$(arg use_nominal_extrinsics)">
         <origin xyz="0.13 0 0.057" rpy="0 ${pi} ${pi}"/>
     </xacro:sensor_d435>

Commit message: keyenece linscanner added

File: staubli_tx90_support/urdf/tx90_macro.xacro (robot description, xacro)
@@ -184,4 +184,30 @@
       </inertial>
   </link>
+  <link name="lj_v7080_frame">
+    <visual>
+      <origin xyz="0 0 0" rpy="0 0 0"/>
+      <geometry>
+        <mesh filename="package://keyence_experimental/meshes/visual/lj_v7080.dae"/>
+      </geometry>
+      <material name="dark grey">
+        <color rgba="0.2 0.2 0.2 1"/>
+      </material>
+    </visual>
+    <collision>
+      <origin xyz="0 0 0" rpy="0 0 0"/>
+      <geometry>
+        <mesh filename="package://keyence_experimental/meshes/collision/lj_v7080.stl"/>
+      </geometry>
+      <material name="dark grey">
+        <color rgba="0.2 0.2 0.2 1"/>
+      </material>
+    </collision>
+  </link>
+  <link name="lj_v7080_optical_frame"/>
+    <joint name="optical_frame" type="fixed">
+      <origin xyz="0 0 0" rpy="0 0 0"/>
+      <parent link="lj_v7080_optical_frame"/>
+      <child link="lj_v7080_frame"/>
+    </joint>
 <!--   <link name="${prefix}PVS_1000_chuck">
     <visual>
@@ -330,8 +356,13 @@
     <!-- ROS-Industrial 'tool0' frame: all-zeros tool frame -->
     <link name="${prefix}tool0" />
-    <joint name="${prefix}flange-tool0" type="fixed">
-      <origin xyz="0.17295 0.0034 0.103" rpy="0 0 0" />
-      <parent link="${prefix}tool_link" />
-      <child link="${prefix}tool0" />
+      <joint name="${prefix}flange-tool0" type="fixed">
+        <origin xyz="0.17295 0.0034 0.103" rpy="0 0 0" />
+        <parent link="${prefix}tool_link" />
+        <child link="${prefix}tool0" />
+      </joint>
+    <joint name="${prefix}tool0-lj_sensor" type="fixed">
+      <origin xyz="-0.037 -0.037 -0.068" rpy="0 ${radians(-90.0)} 0" />   <!--z y x-->
+      <parent link="${prefix}tool0" />
+      <child link="lj_v7080_optical_frame" />
     </joint>
     <!--D435 -->
