Commit message: naming change

File: staubli_tx90_support/urdf/tx90.urdf (robot description, URDF)
Before this commit: robot staubli_tx90, 15 links, 12 joints
Links:
- link tool_link: geometry collision mesh filename=package://tx90_spindle/meshes/base_link.STL; visual mesh filename=package://tx90_spindle/meshes/base_link.STL

File: staubli_tx90_support/urdf/tx90_macro.xacro (robot description, xacro)
@@ -162,5 +162,5 @@
       <origin xyz="0 0 0.001" rpy="0 ${radians(-90.0)} ${radians(180.0)}" />
       <geometry>
-        <mesh filename="package://gripper_2/meshes/base_link.STL" />
+        <mesh filename="package://tx90_spindle/meshes/base_link.STL" />
       </geometry>
       <material name="">
@@ -173,5 +173,5 @@
       <geometry>
         <mesh
-          filename="package://gripper_2/meshes/base_link.STL" />
+          filename="package://tx90_spindle/meshes/base_link.STL" />
       </geometry>
     </collision>

File: tx90_moveit_client/scripts/RL/urdf/tx90.urdf (robot description, URDF)
Before this commit: robot staubli_tx90_gazebo, 12 links, 11 joints
Links:
- link tool_link: geometry collision mesh filename=package://tx90_spindle/meshes/base_link.STL; visual mesh filename=package://tx90_spindle/meshes/base_link.STL

File: tx90_spindle/urdf/gripper_2.urdf (robot description, URDF)
Before this commit: robot gripper_2, 1 links, 0 joints
Links:
- link base_link: geometry collision mesh filename=package://tx90_spindle/meshes/base_link.STL; visual mesh filename=package://tx90_spindle/meshes/base_link.STL
