Commit message: urdf test_bed name changed

File: staubli_tx90_support/urdf/cfrp_macro.xacro (robot description, xacro)
@@ -11,5 +11,5 @@
         <geometry>
           <mesh
-            filename="package://test_bed/meshes/surface_cfrp.STL" />
+            filename="package://tx90_path_planner/meshes/surface_cfrp.STL" />
         </geometry>
       </visual>
@@ -17,5 +17,5 @@
           <geometry>
             <mesh
-              filename="package://test_bed/meshes/surface_cfrp.STL" />
+              filename="package://tx90_path_planner/meshes/surface_cfrp.STL" />
           </geometry>
           <origin xyz="0 0 0" rpy="0 0 0"/>

File: staubli_tx90_support/urdf/tx90.urdf (robot description, URDF)
Before this commit: robot staubli_tx90, 15 links, 12 joints
Links:
- link PVS_1000_chuck: geometry collision mesh filename=package://tx90_path_planner/meshes/PVS_1000_chuck.STL; visual mesh filename=package://tx90_path_planner/meshes/PVS_1000_chuck.dae
- link bed_base: geometry collision mesh filename=package://tx90_path_planner/meshes/base_link.STL; visual mesh filename=package://tx90_path_planner/meshes/base_link.STL

File: staubli_tx90_support/urdf/tx90_macro.xacro (robot description, xacro)
@@ -214,5 +214,5 @@
       <origin xyz="0.0 0.07 0.0"/>
       <geometry>
-        <mesh filename="package://test_bed/meshes/PVS_1000_chuck.dae" />
+        <mesh filename="package://tx90_path_planner/meshes/PVS_1000_chuck.dae" />
       </geometry>
       <material name="light_grey">
@@ -222,5 +222,5 @@
     <collision>
         <geometry>
-            <mesh filename="package://test_bed/meshes/PVS_1000_chuck.STL" />
+            <mesh filename="package://tx90_path_planner/meshes/PVS_1000_chuck.STL" />
         </geometry>
         <origin xyz="0 0 0" rpy="0 0 0"/>
@@ -238,10 +238,10 @@
       </material>
       <geometry>
-        <mesh filename="package://test_bed/meshes/surface_cfrp.STL" />
-      </geometry>
-    </visual>
-    <collision>
-        <geometry>
-            <mesh filename="package://test_bed/meshes/surface_cfrp.STL" />
+        <mesh filename="package://tx90_path_planner/meshes/surface_cfrp.STL" />
+      </geometry>
+    </visual>
+    <collision>
+        <geometry>
+            <mesh filename="package://tx90_path_planner/meshes/surface_cfrp.STL" />
         </geometry>
         <origin xyz="0 0 0" rpy="0 0 0"/>
@@ -267,5 +267,5 @@
       <geometry>
         <mesh
-          filename="package://test_bed/meshes/base_link.STL" />
+          filename="package://tx90_path_planner/meshes/base_link.STL" />
       </geometry>
       <material
@@ -278,5 +278,5 @@
       <geometry>
         <mesh
-          filename="package://test_bed/meshes/base_link.STL" />
+          filename="package://tx90_path_planner/meshes/base_link.STL" />
       </geometry>
     </collision>
