Commit message: normal vector and pcd changed

File: tx90_path_planner/urdf/PVS_1000_chuck.urdf (robot description, URDF)
Before this commit: robot PVS_1000_chuck, 1 links, 0 joints
Links:
- link PVS_1000_chuck: geometry collision mesh filename=package://PVS_1000_chuck/meshes/PVS_1000_chuck.STL; visual mesh filename=package://tx90_path_planner/meshes/PVS_1000_chuck.STL

File: tx90_path_planner/urdf/test_bed.urdf (robot description, URDF)
Before this commit: robot test_bed, 1 links, 0 joints
Links:
- link base_link: geometry collision mesh filename=package://tx90_path_planner/meshes/base_link.STL; visual mesh filename=package://tx90_path_planner/meshes/base_link.STL
